Commit message: ros2 control robo

File: description/lidar.xacro (robot description, xacro)
@@ -1,15 +1,250 @@
 <?xml version="1.0"?>
 <robot xmlns:xacro="http://www.ros.org/wiki/xacro" >
-    <joint name="laser_joint" type="fixed">
+<!-- Support Cylinders -->
+    <joint name="support_cylinder_1_joint" type="fixed">
+        <parent link="chassis"/>
+        <child link="support_cylinder_1"/>
+        <origin xyz="${chassis_length - 0.02} ${chassis_width/2 - 0.02} ${chassis_height}"/>
+    </joint>
+    <link name="support_cylinder_1">
+        <visual>
+            <geometry>
+                <cylinder radius="0.01" length="0.2"/>
+            </geometry>
+            <material name="green"/>
+        </visual>
+        <collision>
+            <geometry>
+                <cylinder radius="0.02" length="0.2"/>
+            </geometry>
+        </collision>
+        <inertial>
+            <mass value="0.1"/>
+            <origin xyz="0 0 0"/>
+            <inertia ixx="0.0001" ixy="0.0" ixz="0.0" iyy="0.0001" iyz="0.0" izz="0.0001"/>
+        </inertial>
+    </link>
+     <joint name="support_cylinder_2_joint" type="fixed">
+        <parent link="chassis"/>
+        <child link="support_cylinder_2"/>
+        <origin xyz="${0.02} ${chassis_width/2 - 0.02} ${chassis_height}"/>
+    </joint>
+    <link name="support_cylinder_2">
+        <visual>
+            <geometry>
+                <cylinder radius="0.01" length="0.2"/>
+            </geometry>
+            <material name="green"/>
+                    </visual>
+        <collision>
+            <geometry>
+                <cylinder radius="0.02" length="0.2"/>
+            </geometry>
+        </collision>
+        <inertial>
+            <mass value="0.1"/>
+            <origin xyz="0 0 0"/>
+            <inertia ixx="0.0001" ixy="0.0" ixz="0.0" iyy="0.0001" iyz="0.0" izz="0.0001"/>
+        </inertial>
+    </link>
+     <joint name="support_cylinder_3_joint" type="fixed">
+        <parent link="chassis"/>
+        <child link="support_cylinder_3"/>
+        <origin xyz="${chassis_length - 0.02} ${-chassis_width/2 + 0.02} ${chassis_height}"/>
+    </joint>
+    <link name="support_cylinder_3">
+        <visual>
+            <geometry>
+                <cylinder radius="0.01" length="0.2"/>
+            </geometry>
+            <material name="green"/>
+                    </visual>
+        <collision>
+            <geometry>
+                <cylinder radius="0.02" length="0.2"/>
+            </geometry>
+        </collision>
+        <inertial>
+            <mass value="0.1"/>
+            <origin xyz="0 0 0"/>
+            <inertia ixx="0.0001" ixy="0.0" ixz="0.0" iyy="0.0001" iyz="0.0" izz="0.0001"/>
+        </inertial>
+    </link>
+     <joint name="support_cylinder_4_joint" type="fixed">
+        <parent link="chassis"/>
+        <child link="support_cylinder_4"/>
+        <origin xyz="${ 0.02} ${-chassis_width/2 + 0.02} ${chassis_height}"/>
+    </joint>
+    <link name="support_cylinder_4">
+        <visual>
+            <geometry>
+                <cylinder radius="0.01" length="0.2"/>
+            </geometry>
+            <material name="green"/>        </visual>
+        <collision>
+            <geometry>
+                <cylinder radius="0.02" length="0.2"/>
+            </geometry>
+        </collision>
+        <inertial>
+            <mass value="0.1"/>
+            <origin xyz="0 0 0"/>
+            <inertia ixx="0.0001" ixy="0.0" ixz="0.0" iyy="0.0001" iyz="0.0" izz="0.0001"/>
+        </inertial>
+    </link>
+    <!-- Tray -->
+    <joint name="tray_joint" type="fixed">
+        <parent link="chassis"/>
+        <child link="tray"/>
+        <origin xyz="${chassis_length /2} 0 ${chassis_height + 0.1}"/>
+    </joint>
+    <link name="tray">
+        <visual>
+            <geometry>
+                <box size="${chassis_length} ${chassis_width} 0.02"/>
+            </geometry>
+            <material name="green"/>
+                    </visual>
+        <collision>
+            <geometry>
+                <box size="${chassis_length} ${chassis_width} 0.02"/>
+            </geometry>
+        </collision>
+        <inertial>
+            <mass value="0.2"/>
+            <origin xyz="0 0 0"/>
+            <inertia ixx="0.0002" ixy="0.0" ixz="0.0" iyy="0.0002" iyz="0.0" izz="0.0002"/>
+        </inertial>
+    </link>
+    <!-- Support Cylinders -->
+    <joint name="support_cylinder_5_joint" type="fixed">
+        <parent link="chassis"/>
+        <child link="support_cylinder_5"/>
+        <origin xyz="${chassis_length - 0.02} ${chassis_width/2 - 0.02} ${chassis_height + 0.12}"/>
+    </joint>
+    <link name="support_cylinder_5">
+        <visual>
+            <geometry>
+                <cylinder radius="0.01" length="0.3"/>
+            </geometry>
+            <material name="green"/>
+                    </visual>
+        <collision>
+            <geometry>
+                <cylinder radius="0.02" length="0.3"/>
+            </geometry>
+        </collision>
+        <inertial>
+            <mass value="0.1"/>
+            <origin xyz="0 0 0"/>
+            <inertia ixx="0.0001" ixy="0.0" ixz="0.0" iyy="0.0001" iyz="0.0" izz="0.0001"/>
+        </inertial>
+    </link>
+     <joint name="support_cylinder_6_joint" type="fixed">
+        <parent link="chassis"/>
+        <child link="support_cylinder_6"/>
+        <origin xyz="${0.02} ${chassis_width/2 - 0.02} ${chassis_height + 0.12}"/>
+    </joint>
+    <link name="support_cylinder_6">
+        <visual>
+            <geometry>
+                <cylinder radius="0.01" length="0.3"/>
+            </geometry>
+            <material name="green"/>
+                    </visual>
+        <collision>
+            <geometry>
+                <cylinder radius="0.02" length="0.3"/>
+            </geometry>
+        </collision>
+        <inertial>
+            <mass value="0.1"/>
+            <origin xyz="0 0 0"/>
+            <inertia ixx="0.0001" ixy="0.0" ixz="0.0" iyy="0.0001" iyz="0.0" izz="0.0001"/>
+        </inertial>
+    </link>
+     <joint name="support_cylinder_7_joint" type="fixed">
+        <parent link="chassis"/>
+        <child link="support_cylinder_7"/>
+        <origin xyz="${chassis_length - 0.02} ${-chassis_width/2 + 0.02} ${chassis_height + 0.12}"/>
+    </joint>
+    <link name="support_cylinder_7">
+        <visual>
+            <geometry>
+                <cylinder radius="0.01" length="0.3"/>
+            </geometry>
+            <material name="green"/>
+                    </visual>
+        <collision>
+            <geometry>
+                <cylinder radius="0.02" length="0.3"/>
+            </geometry>
+        </collision>
+        <inertial>
+            <mass value="0.1"/>
+            <origin xyz="0 0 0"/>
+            <inertia ixx="0.0001" ixy="0.0" ixz="0.0" iyy="0.0001" iyz="0.0" izz="0.0001"/>
+        </inertial>
+    </link>
+     <joint name="support_cylinder_8_joint" type="fixed">
+        <parent link="chassis"/>
+        <child link="support_cylinder_8"/>
+        <origin xyz="${ 0.02} ${-chassis_width/2 + 0.02} ${chassis_height + 0.12}"/>
+    </joint>
+    <link name="support_cylinder_8">
+        <visual>
+            <geometry>
+                <cylinder radius="0.01" length="0.3"/>
+            </geometry>
+            <material name="green"/>
+                    </visual>
+        <collision>
+            <geometry>
+                <cylinder radius="0.02" length="0.3"/>
+            </geometry>
+        </collision>
+        <inertial>
+            <mass value="0.1"/>
+            <origin xyz="0 0 0"/>
+            <inertia ixx="0.0001" ixy="0.0" ixz="0.0" iyy="0.0001" iyz="0.0" izz="0.0001"/>
+        </inertial>
+    </link>
+<!-- Top Tray -->
+    <joint name="top_tray_joint" type="fixed">
+        <parent link="chassis"/>
+        <child link="top_tray"/>
+        <origin xyz="${chassis_length / 2} 0 ${chassis_height + 0.12 + 0.15}"/>
+    </joint>
+    <link name="top_tray">
+        <visual>
+            <geometry>
+                <box size="${chassis_length} ${chassis_width} 0.02"/>
+            </geometry>
+            <material name="green"/>
+                    </visual>
+        <collision>
+            <geometry>
+                <box size="${chassis_length} ${chassis_width} 0.02"/>
+            </geometry>
+        </collision>
+        <inertial>
+            <mass value="0.2"/>
+            <origin xyz="0 0 0"/>
+            <inertia ixx="0.0002" ixy="0.0" ixz="0.0" iyy="0.0002" iyz="0.0" izz="0.0002"/>
+        </inertial>
+    </link>
+    <!-- LIDAR -->
+  <joint name="laser_joint" type="fixed">
         <parent link="chassis"/>
         <child link="laser_frame"/>
-        <origin xyz="0.1 0 0.175" rpy="0 0 0"/>
+        <origin xyz="0.122 0 0.212" rpy="0 0 0"/>
     </joint>
     <link name="laser_frame">
         <visual>
+                 <origin xyz="0 0 0.2"/>
             <geometry>
                 <cylinder radius="0.05" length="0.04"/>
             </geometry>
-            <material name="red"/>
+            <material name="black"/>
         </visual>
         <collision>

File: description/robot.urdf.xacro (robot description, xacro)
@@ -12,3 +12,4 @@
     <!-- <xacro:include filename="ros2_control.xacro" /> -->
     <xacro:include filename="lidar.xacro" />
+        <xacro:include filename="face.xacro" />
 </robot>

File: description/robot_core.xacro (robot description, xacro)
@@ -2,18 +2,24 @@
 <robot xmlns:xacro="http://www.ros.org/wiki/xacro" >
     <xacro:include filename="inertial_macros.xacro"/>
-    <xacro:property name="chassis_length" value="0.335"/>
-    <xacro:property name="chassis_width" value="0.265"/>
-    <xacro:property name="chassis_height" value="0.138"/>
+    <xacro:property name="chassis_length" value="0.22"/>
+    <xacro:property name="chassis_width" value="0.32"/>
+    <xacro:property name="chassis_height" value="0.12"/>
     <xacro:property name="chassis_mass" value="1.0"/>
-    <xacro:property name="wheel_radius" value="0.034"/>
-    <xacro:property name="wheel_thickness" value="0.026"/>
+    <xacro:property name="wheel_radius" value="0.035"/>
+    <xacro:property name="wheel_thickness" value="0.04"/>
     <xacro:property name="wheel_mass" value="0.05"/>
-    <xacro:property name="wheel_offset_x" value="0.226"/>
+    <xacro:property name="wheel_offset_x" value="${chassis_length / 3}"/>
     <xacro:property name="wheel_offset_y" value="0.166"/>
     <xacro:property name="wheel_offset_z" value="0.01"/>
-    <xacro:property name="caster_wheel_radius" value="0.01"/>
-    <xacro:property name="caster_wheel_mass" value="0.01"/>
-    <xacro:property name="caster_wheel_offset_x" value="0.075"/>
-    <xacro:property name="caster_wheel_offset_z" value="${wheel_offset_z - wheel_radius + caster_wheel_radius}"/>
+    <xacro:property name="caster_wheel_left_radius" value="0.035"/>
+    <xacro:property name="caster_wheel_left_mass" value="0.01"/>
+    <xacro:property name="caster_wheel_left_offset_x" value="${chassis_length / 1.5}"/>
+    <xacro:property name="caster_wheel_left_offset_z" value="${wheel_offset_z - wheel_radius + caster_wheel_left_radius}"/>
+    <xacro:property name="caster_wheel_left_offset_y" value="${chassis_width / 3}"/>
+    <xacro:property name="caster_wheel_right_radius" value="0.035"/>
+    <xacro:property name="caster_wheel_right_mass" value="0.01"/>
+    <xacro:property name="caster_wheel_right_offset_x" value="${chassis_length / 1.5}"/>
+    <xacro:property name="caster_wheel_right_offset_z" value="${wheel_offset_z - wheel_radius + caster_wheel_right_radius}"/>
+    <xacro:property name="caster_wheel_right_offset_y" value="${-chassis_width / 3}"/>
     <material name="white">
         <color rgba="1 1 1 1" />
@@ -30,4 +36,7 @@
     <material name="red">
         <color rgba="1 0 0 1"/>
+    </material>
+    <material name="green">
+    <color rgba="0 1 0 1"/>
     </material>
     <!-- BASE LINK -->
@@ -113,14 +122,14 @@
         <material>Gazebo/Blue</material>
     </gazebo>
-    <!-- CASTER WHEEL LINK -->
-    <joint name="caster_wheel_joint" type="fixed">
+    <!-- CASTER WHEEL LINK LEFT-->
+    <joint name="caster_wheel_left_joint" type="fixed">
         <parent link="chassis"/>
-        <child link="caster_wheel"/>
-        <origin xyz="${caster_wheel_offset_x} 0 ${caster_wheel_offset_z}"/>
+        <child link="caster_wheel_left"/>
+        <origin xyz="${caster_wheel_left_offset_x} ${caster_wheel_left_offset_y} ${caster_wheel_left_offset_z}"/>
     </joint>
-    <link name="caster_wheel">
+    <link name="caster_wheel_left">
         <visual>
             <geometry>
-                <sphere radius="${caster_wheel_radius}"/>
+                <sphere radius="${caster_wheel_left_radius}"/>
             </geometry>
             <material name="white"/>
@@ -128,12 +137,39 @@
         <collision>
             <geometry>
-                <sphere radius="${caster_wheel_radius}"/>
+                <sphere radius="${caster_wheel_left_radius}"/>
             </geometry>
         </collision>
-        <xacro:inertial_sphere mass="${caster_wheel_mass}" radius="${caster_wheel_radius}">
+        <xacro:inertial_sphere mass="${caster_wheel_left_mass}" radius="${caster_wheel_left_radius}">
             <origin xyz="0 0 0" rpy="0 0 0"/>
         </xacro:inertial_sphere>
     </link>
-    <gazebo reference="caster_wheel">
+    <gazebo reference="caster_wheel_left">
+        <material>Gazebo/White</material>
+        <mu1 value="0.001"/>
+        <mu2 value="0.001"/>
+    </gazebo>
+    <!-- CASTER WHEEL LINK RIGHT-->
+    <joint name="caster_wheel_right_joint" type="fixed">
+        <parent link="chassis"/>
+        <child link="caster_wheel_right"/>
+        <origin xyz="${caster_wheel_right_offset_x} ${caster_wheel_right_offset_y} ${caster_wheel_right_offset_z}"/>
+    </joint>
+    <link name="caster_wheel_right">
+        <visual>
+            <geometry>
+                <sphere radius="${caster_wheel_right_radius}"/>
+            </geometry>
+            <material name="white"/>
+        </visual>
+        <collision>
+            <geometry>
+                <sphere radius="${caster_wheel_right_radius}"/>
+            </geometry>
+        </collision>
+        <xacro:inertial_sphere mass="${caster_wheel_right_mass}" radius="${caster_wheel_right_radius}">
+            <origin xyz="0 0 0" rpy="0 0 0"/>
+        </xacro:inertial_sphere>
+    </link>
+    <gazebo reference="caster_wheel_right">
         <material>Gazebo/White</material>
         <mu1 value="0.001"/>

File: description/ros2_control.xacro (robot description, xacro)
@@ -1,5 +1,33 @@
 <?xml version="1.0"?>
 <robot xmlns:xacro="http://www.ros.org/wiki/xacro">
-    <ros2_control name="GazeboSystem" type="system">
+    <ros2_control name="RealRobot" type="system">
+            <hardware>
+                <plugin>diffdrive_arduino/DiffDriveArduino</plugin>
+                <param name="left_wheel_name">left_wheel_joint</param>
+                <param name="right_wheel_name">right_wheel_joint</param>
+                <param name="loop_rate">30</param>
+                <param name="device">/dev/ttyACM0</param>
+                <param name="baud_rate">57600</param>
+                <param name="timeout">1000</param>
+                <param name="enc_counts_per_rev">12600</param>
+            </hardware>
+            <joint name="left_wheel_joint">
+                <command_interface name="velocity">
+                    <param name="min">-10</param>
+                    <param name="max">10</param>
+                </command_interface>
+                <state_interface name="velocity"/>
+                <state_interface name="position"/>
+            </joint>
+            <joint name="right_wheel_joint">
+                <command_interface name="velocity">
+                    <param name="min">-10</param>
+                    <param name="max">10</param>
+                </command_interface>
+                <state_interface name="velocity"/>
+                <state_interface name="position"/>
+            </joint>
+        </ros2_control>
+    <!-- <ros2_control name="GazeboSystem" type="system">
         <hardware>
             <plugin>gazebo_ros2_control/GazeboSystem</plugin>
@@ -21,5 +49,5 @@
             <state_interface name="position"/>
         </joint>
-    </ros2_control>
+    </ros2_control> -->
     <gazebo>
         <plugin name="gazebo_ros2_control" filename="libgazebo_ros2_control.so">
